File: Circuit/KiCad/CWKeyer/CWKeyer.kicad_sch (KiCad schematic)
At the start: 6 parts, among them J1 Conn_01x15_Pin

Commit message: PCB Update
Parts:
- removed J1: Conn_01x15_Pin, Connector_PinSocket_2.54mm:PinSocket_1x15_P2.54mm_Vertical, symbol Connector:Conn_01x15_Pin
- removed J2: (no value), Connector_PinSocket_2.54mm:PinSocket_1x15_P2.54mm_Vertical, symbol Connector:Conn_01x15_Pin
- removed R1: 10k, PCM_SL_Devices:Potentiometer_RM065, symbol PCM_SL_Devices:potentiometer_RM065
- added A1: Lolin_NodeMCU_ESP8266_V3, PCM_SL_Development_Boards:Lolin_NodeMCU_ESP8266, symbol PCM_SL_Development_Board:Lolin_NodeMCU_ESP8266_V3
- added J1: Encoder, Connector_PinHeader_2.54mm:PinHeader_1x05_P2.54mm_Vertical, symbol Connector:Conn_01x05_Pin
- added J2: AudioIn, Connector_Audio:Jack_3.5mm_PJ320E_Horizontal, symbol Connector_Audio:AudioJack3_Ground
- added J3: Headphone, Connector_Audio:Jack_3.5mm_PJ320E_Horizontal, symbol Connector_Audio:AudioJack3_Ground
- added J4: Keyer, Connector_Audio:Jack_3.5mm_PJ320E_Horizontal, symbol Connector_Audio:AudioJack3_Ground
- added RV1: R_Potentiometer, Potentiometer_THT:Potentiometer_Piher_PT-10-V10_Vertical, symbol Device:R_Potentiometer
Connections:
- net at C1.1, R2.2, R3.1: now also A1.16 (ADC0)
- net at R3.2: now also A1.29 (GND), J1.5 (Pin_5), J2.S, J3.S, J4.S
- net at R2.1: now also A1.1 (3V3)
- net at C1.2: now also J2.R, J2.T
- new net: A1.10 (3V3), J1.4 (Pin_4)
- new net: A1.11 (D4/GPIO2/TX1), J1.1 (Pin_1)
- new net: A1.12 (D3/GPIO0), J1.2 (Pin_2)
- new net: A1.15 (D0/GPIO16/WAKE), J1.3 (Pin_3)
- new net: A1.17 (GND), RV1.3
- new net: A1.6 (D7/GPIO13/MOSI/RX2), J4.R
- new net: A1.7 (D6/GPIO12/MISO), J4.T
- new net: A1.8 (D5/GPIO14/SCLK), RV1.1
- new net: J3.R, J3.T, RV1.2
Other:
- note removed: "ESP8266"
