File: Circuit/KiCad/CWKeyer/CWKeyer.kicad_pcb (KiCad board)
At the start: 2 copper layers, 2 parts, among them J1 Conn_01x15_Pin, J2 Conn_01x15_Pin

Commit message: PCB Update
Parts:
- added A1: Lolin_NodeMCU_ESP8266_V3, PCM_SL_Development_Boards:Lolin_NodeMCU_ESP8266, F.Cu at (92.7, 73.7)
- added C1: 100nF_Ceramic, Capacitor_THT:C_Disc_D5.0mm_W2.5mm_P2.50mm, F.Cu at (119.4, 55.9)
- added J3: Headphone, Connector_Audio:Jack_3.5mm_PJ320E_Horizontal, F.Cu at (173.3, 63.5)
- added J4: Keyer, Connector_Audio:Jack_3.5mm_PJ320E_Horizontal, F.Cu at (174.5, 93.8)
- added R2: 10k, Resistor_THT:R_Axial_DIN0207_L6.3mm_D2.5mm_P10.16mm_Horizontal, F.Cu at (129.5, 68.6)
- added R3: 10k, Resistor_THT:R_Axial_DIN0207_L6.3mm_D2.5mm_P10.16mm_Horizontal, F.Cu at (119.4, 63.5)
- added RV1: R_Potentiometer, Potentiometer_THT:Potentiometer_Piher_PT-10-V10_Vertical, F.Cu at (149.9, 86.3)
- J1: value Conn_01x15_Pin -> Encoder; footprint Connector_PinSocket_2.54mm:PinSocket_1x15_P2.54mm_Vertical -> Connector_PinHeader_2.54mm:PinHeader_1x05_P2.54mm_Vertical
- J2: value Conn_01x15_Pin -> AudioIn; footprint Connector_PinSocket_2.54mm:PinSocket_1x15_P2.54mm_Vertical -> Connector_Audio:Jack_3.5mm_PJ320E_Horizontal
- moved J1 132.0 mm to (184.1, 83.1)
- moved J2 92.9 mm to (173.3, 48.3), turned to -90 degrees
Connections:
- J1 pad 1: unconnected-(J1-Pin_1-Pad1) -> Net-(A1-D4/GPIO2/TX1)
- J1 pad 2: unconnected-(J1-Pin_2-Pad2) -> Net-(A1-D3/GPIO0)
- J1 pad 3: unconnected-(J1-Pin_3-Pad3) -> Net-(A1-D0/GPIO16/WAKE)
- J1 pad 4: unconnected-(J1-Pin_4-Pad4) -> Net-(J1-Pin_4)
- J1 pad 5: unconnected-(J1-Pin_5-Pad5) -> Net-(J1-Pin_5)
Routing:
- net Net-(A1-ADC0): track 0.00 -> 3.45 mm
